File: electronics/07-comms.kicad_sch (KiCad schematic)
At the start: 19 parts, among them J701 Module BLE (HM-11 / ESP32-C3), J702 Embase ESC (signal), J703 Puissance turbine (XT30), Q701 SI2301CDS, Q702 AO3400A, U701 W25Q128JVSIQ

Commit message: Passe le microcontrôleur en LQFP144 et lit les deux courants au même instant
Le LQFP100 avait ses seize entrées ADC prises — douze voies de ligne, trois
de télémétrie, une sortie de multiplexeur — et c'est ce multiplexeur qui
posait le vrai problème : il interdisait par construction de lire les deux
courants moteur ensemble. On lisait un moteur, on commutait, on attendait
l'établissement, on lisait l'autre. Le STM32H723ZGT6 en LQFP144 place
PF11 sur ADC1_INP2 et PF13 sur ADC2_INP2 : même numéro de voie sur deux
convertisseurs, donc une lecture simultanée en mode double, et le 74HC4051
disparaît de la carte.

Le brochage étant donné par nom de port et non par numéro de broche, le
passage a coûté deux affectations sur quatre-vingt-sept. Une affectation est
un choix de port — PA0 porte la voie de ligne 00 — jamais un choix de patte.
Une table numérotée aurait demandé de recopier 144 lignes à la main, et une
erreur de brochage ne se voit pas à l'ERC.

Ajoute une huitième feuille, les témoins de ligne. Ce qu'on regarde pendant
un essai n'est pas un témoin d'état générique, c'est ce que voit la
moustache : une LED par capteur, à l'aplomb du capteur qu'elle rapporte, et
un capteur borgne se voit avant la course plutôt qu'après. Le rapport
cyclique suit le signal, sinon rien ne dirait si la ligne est au bord ou au
centre du trait. PCA9685 à l'adresse 0x40 sur I²C2, 52 octets par rafale
soit 1,2 ms à 400 kHz, en DMA hors de la boucle rapide.

Remplace l'interrupteur à glissière par une mise sous tension à bouton
poussoir : une impulsion amorce, le microcontrôleur se tient lui-même, et
c'est lui qui coupe. La glissière demandait une place au bord de carte que
le pack, l'équilibrage et les fils de l'ESC ont fini par prendre — et elle
ne savait pas éteindre proprement, couper le 3,3 V sous les pieds du
firmware n'ayant jamais rien écrit dans la flash.

Ajoute au générateur le contrôle qui manquait : deux extrémités de nets
différents au même point. Il a fallu qu'il relie B+ à B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
Parts:
- removed J703: Puissance turbine (XT30), Connector_AMASS:AMASS_XT30U-M_1x02_P5.0mm_Vertical, symbol Connector_Generic:Conn_01x02
- added J103: MultiStar 10A (debout), Pacabot:ESC_Multistar_10A, symbol Connector_Generic:Conn_01x02
- C701, C703, C705: footprint Capacitor_SMD:C_0603_1608Metric -> Capacitor_SMD:C_0402_1005Metric; Dielectric (none) -> X7R; Voltage (none) -> 25V
- C702: value 10uF/10V -> 10uF; Dielectric (none) -> X5R; Voltage (none) -> 10V
- C704: value 220uF/16V -> 220uF; footprint Capacitor_SMD:CP_Elec_8x10 -> Capacitor_SMD:CP_Elec_6.3x7.7; Dielectric (none) -> ALU; Voltage (none) -> 10V
- J701: value Module BLE (HM-11 / ESP32-C3) -> Module OTA (ESP32-C3); footprint Connector_PinHeader_2.54mm:PinHeader_1x06_P2.54mm_Vertical -> Connector_PinHeader_2.54mm:PinHeader_1x04_P2.54mm_Vertical; symbol Connector_Generic:Conn_01x06 -> Connector_Generic:Conn_01x04
- J702: value Embase ESC (signal) -> Signal ESC (coudee); footprint Connector_PinHeader_2.54mm:PinHeader_1x03_P2.54mm_Vertical -> Connector_PinHeader_2.54mm:PinHeader_1x01_P2.54mm_Horizontal; symbol Connector_Generic:Conn_01x03 -> Connector_Generic:Conn_01x01
- R701, R702, R703, R704, R705, R706, R707: footprint Resistor_SMD:R_0603_1608Metric -> Resistor_SMD:R_0402_1005Metric; Power (none) -> 63mW
Connections:
- net ESC_SIG: now also J702.1 (Pin_1); no longer J702.3 (Pin_3)
- net GND: now also J103.2 (Pin_2); no longer J702.1 (Pin_1)
- net VBAT: now also J103.1 (Pin_1)
- no-connect marks 3 -> 0
Other:
- note added: "Calibre : la turbine tire 11 A a 8,4 V, mais elle est ici sur VBAT (5,0 a 7,3 V) et le courant d une helice suit le carre de la tension : 11 x (6,4/8,4)^2 = 6,4 A sur le plateau LiFePO4. Les 10 A continus du MultiStar tiennent donc, avec 15 A de crete a la mise en rotation. A verifier a la pince amperemetrique au premier essai en charge."
- note added: "PA8 haut = module alimente. Grille rappelee au rail par R703 : MCU eteint ou GPIO en haute impedance, le module reste hors tension. Module conseille : ESP32-C3 SuperMini - OTA par WiFi natif (rapide), pont UART 921600 Bd vers le STM32. Un HM-11 BLE 4.0 plafonne a 2-3 ko/s : 2 a 4 min pour 256 ko de firmware. Broche 3 = RX du module, broche 4 = TX : a recroiser selon la serigraphie."
- note added: "Puissance prise sur VBAT en amont des ponts moteurs, avec son propre decouplage. Rampe la consigne : une montee en regime brutale fait chuter VBAT et peut faire redemarrer le MCU en pleine ligne droite. L armement de l ESC fait partie de la sequence de pre-depart, pas du demarrage du firmware. F101 12 A et les deux AO4407A en parallele de la feuille 01 laissent la marge."
- note added: "Turnigy MultiStar 10A BLHeli-S (Opto) : 22 x 12 mm, 5,1 g, 10 A continu / 15 A crete. Il est DEBOUT sur sa tranche cote entree de puissance, ses deux fils soudes dans J103 et un collier au corps : 12 x 5 mm d emprise pour 22 mm de haut. Aucun connecteur ne s intercale sur le courant de la turbine."
- note added: "Une seule broche, et COUDEE : le variateur est debout juste a cote, son fil de commande arrive a plat le long de la carte. Le cordon trois fils est coupe - le fil central (BEC) sort 5 ou 6 V sur la plupart des variateurs et emporterait le rail 3,3 V, et le fil de masse est inutile puisque le meme cuivre revient par le fil noir de puissance soude en J103, a quelques millimetres de la."
- note removed: "Broche 2 = BEC. La plupart des ESC y sortent 5 ou 6 V : reliee au rail 3,3 V elle emporte toute la carte. Elle reste donc explicitement non connectee."
- note removed: "PA8 haut = module alimente. Grille rappelee au rail par R703 : MCU eteint ou GPIO en haute impedance, le module reste hors tension. Broche 3 = RX du module, broche 4 = TX du module : a recroiser selon la serigraphie du module retenu."
- note removed: "Puissance prise sur VBAT en amont des ponts moteurs, avec son propre decouplage. Rampe la consigne : une montee en regime brutale fait chuter VBAT et peut faire redemarrer le MCU en pleine ligne droite. L armement de l ESC fait partie de la sequence de pre-depart, pas du demarrage du firmware. La turbine peut tirer 5 a 15 A : verifier que le fusible F101, l interrupteur J105 et le MOSFET Q102 de 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"

Commit message: Replace la carte autour de ses chaînes analogiques et y intègre le pack commun et l'ESC
Le placement du 4 septembre rangeait les pièces par zone. Celui-ci part des
nets et des vraies pastilles, et affecte chaque condensateur à une broche
plutôt qu'à une couronne autour du boîtier. Le STM32 pivote de 180° sur son
centre pour tourner son côté analogique vers la barrette. Chaque station
laser reçoit son propre TLV9064 (U504 s'ajoute pour la station L), et la
liaison photodiode → TIA tombe de 34, 56 et 69 mm à 3,1, 7,4 et 2,9 mm. La
boucle de retour du TIA passe de 140–150 mm à 3,55. Cinq découplages
suivent : C568, C569/C570 sur VREF_RX, C223/C224 sur VBAT du MCU et C351
sur VREF_MOT du pont droit.

`layout.py`, `layout_fit.json` et `place_pcb.py --reset` ne décrivent plus
cette carte. Le README le dit en tête, et les nouveaux outils partent du
PCB courant, jamais de l'ancienne table. `audit_placement_geometry.py` relit
les courtyards orientés et les contrôle sous Shapely, `placement_metrics.py`
et `preview_analog_paths.py` mesurent distances et couloirs sans poser une
piste. `refine_placement.py` calcule la table, `apply_refined_placement.py`
l'écrit en vérifiant verrous et UUID : il ne se rejoue pas après une
retouche à la main.

L'alimentation change de nature. Le pack LiFePO4 et son ESC sur VBAT
laissent place à un pack 2S commun, chimie encore à choisir, que la carte,
les moteurs et la turbine partagent. Une seule prise MR30 à trois contacts
porte GND, point milieu et VPACK, et remplace XT30 + JST-XH. L'ESC devient
un EMAX Bullet 12A (12 A continu, 15 A crête, sans BEC) sur VPACK brut,
monté debout sur J103. J104 et J702 disparaissent. ESC103 et M703 sont des
symboles hors carte : les phases moteur ne reçoivent aucun pad fictif, et
le module ne compte qu'une fois dans la nomenclature. R107 passe de 10 à
47 Ω pour ramener l'équilibrage à 88 mA et 0,36 W, sous le watt de son
boîtier 2512. La recharge reste inhibée par défaut matériel tant que
cellules, profil et fir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
Parts:
- removed J702: Signal ESC (coudee), Connector_PinHeader_2.54mm:PinHeader_1x01_P2.54mm_Horizontal, symbol Connector_Generic:Conn_01x01
- added ESC103: EMAX Bullet 12A EMX-SC-1873, Pacabot:EMAX_Bullet_12A_Vertical_3Pin_PROTOTYPE, symbol Pacabot:EMAX_Bullet_12A_EMX_SC_1873
- added M703: Turbine / fils hors PCB, symbol Pacabot:Turbine_3Phase_Offboard
- C704: symbol Device:C -> Device:C_Polarized; Voltage 10V -> 16V
- J103: value MultiStar 10A (debout) -> Montage vertical ESC (prototype); footprint Pacabot:ESC_Multistar_10A -> Pacabot:EMAX_Bullet_12A_Vertical_3Pin_PROTOTYPE; symbol Connector_Generic:Conn_01x02 -> Pacabot:ESC_Vertical_Mount3; Mechanical_status (none) -> PROTOTYPE - measure physical ESC before fabrication; Power_pins (none) -> Solid copper diameter 1.20 mm; holes 1.40 mm; pads 3.00 mm; now left out of the parts list
Connections:
- net ESC_SIG: now also J103.2 (SIGNAL), ESC103.2 (SIGNAL)
- net GND: now also J103.1 (GND_POWER), ESC103.1 (GND_POWER); no longer J103.2 (Pin_2)
- net VBAT renamed VPACK
- net VPACK: now also J103.3 (+BATT), ESC103.3 (+BATT); no longer J103.1 (Pin_1)
- new net ESC_PHASE_A: ESC103.4 (MOTOR_A), M703.1 (A)
- new net ESC_PHASE_B: ESC103.5 (MOTOR_B), M703.2 (B)
- new net ESC_PHASE_C: ESC103.6 (MOTOR_C), M703.3 (C)
Other:
- note added: "J103 : trois pins sur la carte. ESC103 et M703 : circuit externe, exclus du PCB. Les sorties moteur ne passent pas dans le cuivre de la carte. PCB ESC 11 x 15 mm; montage vertical avec soutien isolant a realiser. Entraxes et epaisseurs estimes sur photos : valider sur la piece avant fabrication."
- note added: "Turbine : EMAX Bullet 12A EMX-SC-1873 / BLHeli-S / sans BEC"
- note added: "VPACK = batterie brute : ESC sous tension tant que le pack est branche. F101 et le bouton coupent la carte / traction, pas la branche ESC. Pack commun 2S : protection generale et profil de charge a definir avec les cellules. Petit GND logique et gros GND puissance : continuite a mesurer; sinon 4e liaison requise."
- note removed: "Calibre : la turbine tire 11 A a 8,4 V, mais elle est ici sur VBAT (5,0 a 7,3 V) et le courant d une helice suit le carre de la tension : 11 x (6,4/8,4)^2 = 6,4 A sur le plateau LiFePO4. Les 10 A continus du MultiStar tiennent donc, avec 15 A de crete a la mise en rotation. A verifier a la pince amperemetrique au premier essai en charge."
- note removed: "Puissance prise sur VBAT en amont des ponts moteurs, avec son propre decouplage. Rampe la consigne : une montee en regime brutale fait chuter VBAT et peut faire redemarrer le MCU en pleine ligne droite. L armement de l ESC fait partie de la sequence de pre-depart, pas du demarrage du firmware. F101 12 A et les deux AO4407A en parallele de la feuille 01 laissent la marge."
- note removed: "Turbine d appui - l ESC est autonome, la carte ne lui envoie qu une consigne"
- note removed: "Turnigy MultiStar 10A BLHeli-S (Opto) : 22 x 12 mm, 5,1 g, 10 A continu / 15 A crete. Il est DEBOUT sur sa tranche cote entree de puissance, ses deux fils soudes dans J103 et un collier au corps : 12 x 5 mm d emprise pour 22 mm de haut. Aucun connecteur ne s intercale sur le courant de la turbine."
- note removed: "Une seule broche, et COUDEE : le variateur est debout juste a cote, son fil de commande arrive a plat le long de la carte. Le cordon trois fils est coupe - le fil central (BEC) sort 5 ou 6 V sur la plupart des variateurs et emporterait le rail 3,3 V, et le fil de masse est inutile puisque le meme cuivre revient par le fil noir de puissance soude en J103, a quelques millimetres de la."
- moved on the sheet: C705, R707
