File: electronics/UsainBot.kicad_pcb (KiCad board)
At the start: 4 copper layers, 155 x 164.9 mm, 335 parts, among them J101 TYPE-C-31-M-12, J102 Pack 2S - puissance, J103 MultiStar 10A (debout), J104 Pack 2S - equilibrage, J201 TC2030-IDC-FP, J301 Moteur Faulhaber + IE2, J351 Moteur Faulhaber + IE2, J601 OLED SSD1306 I2C, J701 Module OTA (ESP32-C3), J702 Signal ESC (coudee), M1 Faulhaber 1524T006SR + IE2 + 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, M2 Faulhaber 1524T006SR + IE2 + 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, M3 Turbine_EDF27_dessus, Q101 AO3400A, Q102 AO4407A, Q103 AO4407A, Q104 AO3400A, Q401 AO3400A, Q402 AO3400A, Q501 AO3400A, Q521 AO3400A, Q541 AO3400A, Q601 AO3400A, Q602 AO3400A, Q701 SI2301CDS, Q702 AO3400A, SW101 MARCHE / ARRET, SW601 SKRHABE010, SW602 START, SW603 RESET, U101 USBLC6-2SC6, U102 BQ25887RGER, U103 TPS62933DRLR, U105 PCA9685PW, U201 STM32H723ZGT6, U301 DRV8874PWPR, U351 DRV8874PWPR, U401 ITR8307/S17/TR8, U402 ITR8307/S17/TR8, U403 ITR8307/S17/TR8, U404 ITR8307/S17/TR8, U405 ITR8307/S17/TR8, U406 ITR8307/S17/TR8, U407 ITR8307/S17/TR8, U408 ITR8307/S17/TR8, U409 ITR8307/S17/TR8, U410 ITR8307/S17/TR8, U411 ITR8307/S17/TR8, U412 ITR8307/S17/TR8, U501 TLV9064, U502 TLV9064, U503 LSM6DSOTR, U701 W25Q128JVSIQ, Y201 25 MHz / 10 ppm

Commit message: Replace la carte autour de ses chaînes analogiques et y intègre le pack commun et l'ESC
Le placement du 4 septembre rangeait les pièces par zone. Celui-ci part des
nets et des vraies pastilles, et affecte chaque condensateur à une broche
plutôt qu'à une couronne autour du boîtier. Le STM32 pivote de 180° sur son
centre pour tourner son côté analogique vers la barrette. Chaque station
laser reçoit son propre TLV9064 (U504 s'ajoute pour la station L), et la
liaison photodiode → TIA tombe de 34, 56 et 69 mm à 3,1, 7,4 et 2,9 mm. La
boucle de retour du TIA passe de 140–150 mm à 3,55. Cinq découplages
suivent : C568, C569/C570 sur VREF_RX, C223/C224 sur VBAT du MCU et C351
sur VREF_MOT du pont droit.

`layout.py`, `layout_fit.json` et `place_pcb.py --reset` ne décrivent plus
cette carte. Le README le dit en tête, et les nouveaux outils partent du
PCB courant, jamais de l'ancienne table. `audit_placement_geometry.py` relit
les courtyards orientés et les contrôle sous Shapely, `placement_metrics.py`
et `preview_analog_paths.py` mesurent distances et couloirs sans poser une
piste. `refine_placement.py` calcule la table, `apply_refined_placement.py`
l'écrit en vérifiant verrous et UUID : il ne se rejoue pas après une
retouche à la main.

L'alimentation change de nature. Le pack LiFePO4 et son ESC sur VBAT
laissent place à un pack 2S commun, chimie encore à choisir, que la carte,
les moteurs et la turbine partagent. Une seule prise MR30 à trois contacts
porte GND, point milieu et VPACK, et remplace XT30 + JST-XH. L'ESC devient
un EMAX Bullet 12A (12 A continu, 15 A crête, sans BEC) sur VPACK brut,
monté debout sur J103. J104 et J702 disparaissent. ESC103 et M703 sont des
symboles hors carte : les phases moteur ne reçoivent aucun pad fictif, et
le module ne compte qu'une fois dans la nomenclature. R107 passe de 10 à
47 Ω pour ramener l'équilibrage à 88 mA et 0,36 W, sous le watt de son
boîtier 2512. La recharge reste inhibée par défaut matériel tant que
cellules, profil et fir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
Parts:
- removed J104: Pack 2S - equilibrage, JST_XH_B3B-XH-A_1x03_P2.50mm_Vertical
- removed J702: Signal ESC (coudee), PinHeader_1x01_P2.54mm_Horizontal
- added C223: 100nF, Capacitor_SMD:C_0402_1005Metric, F.Cu at (141.4, 220.9)
- added C224: 1uF, Capacitor_SMD:C_0402_1005Metric, F.Cu at (143.0, 222.5)
- added C351: 100nF, Capacitor_SMD:C_0402_1005Metric, F.Cu at (208.4, 131.8)
- added C568: 100nF, Capacitor_SMD:C_0402_1005Metric, F.Cu at (179.7, 167.7)
- added C569: 100nF, Capacitor_SMD:C_0402_1005Metric, F.Cu at (169.3, 189.2)
- added C570: 100nF, Capacitor_SMD:C_0402_1005Metric, F.Cu at (182.4, 165.5)
- added U504: TLV9064, Package_SO:TSSOP-14_4.4x5mm_P0.65mm, F.Cu at (179.4, 172.5)
- BZ601: footprint MagneticBuzzer_ProSignal_ABI-009-RC -> Buzzer_Beeper:MagneticBuzzer_ProSignal_ABI-009-RC
- C101: footprint C_0603_1608Metric -> Capacitor_SMD:C_0603_1608Metric
- C102, C103, C106, C107, C111, C112: footprint C_1210_3225Metric -> Capacitor_SMD:C_1210_3225Metric
- C104, C110, C113, C114, C115, C118, C120, C121, C201, C202, C203, C204, C205, C207, C208, C209, C210, C211, C214, C215, C216, C217, C218, C219, C220, C221, C222, C303, C305, C306, C353, C355, C501, C502, C503, C504, C505, C521, C522, C523, C524, C525, C541, C542, C543, C544, C545, C561, C562, C563, C564, C566, C567, C601, C602, C603, C604, C605, C606, C607, C701, C703, C705: footprint C_0402_1005Metric -> Capacitor_SMD:C_0402_1005Metric
- C105, C108, C116, C117, C119, C206, C212, C213, C307, C565, C702: footprint C_0805_2012Metric -> Capacitor_SMD:C_0805_2012Metric
- C109, C704: footprint CP_Elec_6.3x7.7 -> Capacitor_SMD:CP_Elec_6.3x7.7
- C122, C123, C124, C301, C302, C308, C309, C352, C356, C358, C359, C401, C402, C403, C404, C405, C406, C407, C408, C409, C410, C411, C412: footprint C_0402_1005Metric -> Capacitor_SMD:C_0402_1005Metric; moved to F.Cu
- C304: footprint CP_EIA-7343-20_Kemet-V -> Capacitor_Tantalum_SMD:CP_EIA-7343-20_Kemet-V
- C354: footprint CP_EIA-7343-20_Kemet-V -> Capacitor_Tantalum_SMD:CP_EIA-7343-20_Kemet-V; moved to F.Cu
- C357: footprint C_0805_2012Metric -> Capacitor_SMD:C_0805_2012Metric; moved to F.Cu
- D101, D401, D402, D403, D404, D405, D406, D407, D408, D409, D410, D411, D412, D606, D701: footprint LED_0603_1608Metric -> LED_SMD:LED_0603_1608Metric
- D102: footprint D_SMB -> Diode_SMD:D_SMB
- D106: footprint D_SOD-323 -> Diode_SMD:D_SOD-323; moved to F.Cu
- D503, D504, D523, D524, D543, D544, D601, D610: footprint D_SOD-323 -> Diode_SMD:D_SOD-323
- D608: value rouge - arriere -> rouge - coin arriere gauche; footprint LED_0603_1608Metric -> LED_SMD:LED_0603_1608Metric
- D609: value rouge - arriere -> rouge - coin arriere droit; footprint LED_0603_1608Metric -> LED_SMD:LED_0603_1608Metric
- F101: footprint R_1206_3216Metric -> Resistor_SMD:R_1206_3216Metric
- FB101: footprint L_0805_2012Metric -> Inductor_SMD:L_0805_2012Metric
- J101: footprint USB_C_Receptacle_HRO_TYPE-C-31-M-12 -> Connector_USB:USB_C_Receptacle_HRO_TYPE-C-31-M-12
- J102: value Pack 2S - puissance -> Pack 2S - AMASS MR30; footprint AMASS_XT30U-M_1x02_P5.0mm_Vertical -> Pacabot:AMASS_MR30PB-M_1x03_P3.50mm_Vertical
- J103: value MultiStar 10A (debout) -> Montage vertical ESC (prototype); footprint Pacabot:ESC_Multistar_10A -> Pacabot:EMAX_Bullet_12A_Vertical_3Pin_PROTOTYPE
- J201: footprint Tag-Connect_TC2030-IDC-FP_2x03_P1.27mm_Vertical -> Connector:Tag-Connect_TC2030-IDC-FP_2x03_P1.27mm_Vertical
- J301, J351: footprint TE_Micro-MaTch_215079-6_2x03_P1.27mm_Vertical -> Connector_TE-Connectivity:TE_Micro-MaTch_215079-6_2x03_P1.27mm_Vertical
- J601: footprint OLED_096_I2C -> Pacabot:OLED_096_I2C
- J701: footprint PinHeader_1x04_P2.54mm_Vertical -> Connector_PinHeader_2.54mm:PinHeader_1x04_P2.54mm_Vertical
- L101: footprint L_Taiyo-Yuden_NR-30xx -> Inductor_SMD:L_Taiyo-Yuden_NR-30xx
- L102: footprint L_Taiyo-Yuden_NR-40xx -> Inductor_SMD:L_Taiyo-Yuden_NR-40xx
- Q101, Q104: footprint SOT-23 -> Package_TO_SOT_SMD:SOT-23; moved to F.Cu
- Q102, Q103: footprint SOIC-8_3.9x4.9mm_P1.27mm -> Package_SO:SOIC-8_3.9x4.9mm_P1.27mm
- Q401, Q402, Q501, Q521, Q541, Q601, Q602, Q701, Q702: footprint SOT-23 -> Package_TO_SOT_SMD:SOT-23
- R101, R102, R106, R110, R114, R115, R116, R117, R118, R119, R120, R201, R202, R203, R204, R441, R442, R443, R444, R445, R446, R447, R448, R449, R450, R451, R452, R453, R454, R455, R456, R501, R502, R503, R504, R505, R506, R507, R508, R521, R522, R523, R524, R525, R526, R527, R528, R541, R542, R543, R544, R545, R546, R547, R548, R561, R562, R563, R564, R601, R602, R603, R604, R605, R606, R607, R608, R609, R610, R615, R617, R618, R619, R620, R701, R702, R703, R704, R705, R706, R707: footprint R_0402_1005Metric -> Resistor_SMD:R_0402_1005Metric
- R103, R104, R105, R108, R109, R111, R112, R113, R124, R125, R126, R127, R128, R301, R302, R303, R304, R305, R306, R307, R308, R309, R310, R353, R354, R355, R356, R357, R358, R359, R360, R401, R402, R403, R404, R405, R406, R407, R408, R409, R410, R411, R412, R421, R422, R423, R424, R425, R426, R427, R428, R429, R430, R431, R432: footprint R_0402_1005Metric -> Resistor_SMD:R_0402_1005Metric; moved to F.Cu
- R107: value 10R -> 47R; footprint R_2512_6332Metric -> Resistor_SMD:R_2512_6332Metric
- SW101, SW602, SW603: footprint SW_SPST_B3U-1000P -> Button_Switch_SMD:SW_SPST_B3U-1000P
- SW601: footprint SKRHABE010 -> Pacabot:SKRHABE010
- TM501, TM521, TM541: footprint Telemetry_Duo_Coude -> Pacabot:Telemetry_Duo_Coude
- U101: footprint SOT-23-6 -> Package_TO_SOT_SMD:SOT-23-6
- U102: footprint HVQFN-24-1EP_4x4mm_P0.5mm_EP2.6x2.6mm_ThermalVias -> Package_DFN_QFN:HVQFN-24-1EP_4x4mm_P0.5mm_EP2.6x2.6mm_ThermalVias
- U103: footprint SOT-583-8 -> Package_TO_SOT_SMD:SOT-583-8
- U105: footprint TSSOP-28_4.4x9.7mm_P0.65mm -> Package_SO:TSSOP-28_4.4x9.7mm_P0.65mm; moved to F.Cu
- U201: footprint LQFP-144_20x20mm_P0.5mm -> Package_QFP:LQFP-144_20x20mm_P0.5mm
- U301, U351: footprint HTSSOP-16-1EP_4.4x5mm_P0.65mm_EP3.4x5mm -> Package_SO:HTSSOP-16-1EP_4.4x5mm_P0.65mm_EP3.4x5mm
- U401, U402, U403, U404, U405, U406, U407, U408, U409, U410, U411, U412: value ITR8307/S17/TR8 -> ITR8307/S17/TR8(B); footprint ITR8307_dessous -> Pacabot:ITR8307_S17_TR8_Bottom
- U501, U502: footprint TSSOP-14_4.4x5mm_P0.65mm -> Package_SO:TSSOP-14_4.4x5mm_P0.65mm
- U503: footprint LGA-14_3x2.5mm_P0.5mm_LayoutBorder3x4y -> Package_LGA:LGA-14_3x2.5mm_P0.5mm_LayoutBorder3x4y
- U701: footprint SOIC-8_5.3x5.3mm_P1.27mm -> Package_SO:SOIC-8_5.3x5.3mm_P1.27mm
- Y201: footprint Crystal_SMD_3225-4Pin_3.2x2.5mm -> Crystal:Crystal_SMD_3225-4Pin_3.2x2.5mm
- moved C302 117.9 mm to (161.4, 228.1), turned to -135 degrees
- moved R308 116.5 mm to (162.2, 228.9), turned to 45 degrees
- moved R127 110.3 mm to (139.2, 217.3), turned to 45 degrees
- moved R358 107.5 mm to (163.6, 227.5), turned to 45 degrees
- moved C352 103.4 mm to (162.8, 226.7), turned to -135 degrees
- moved C122 101.2 mm to (140.4, 214.1), turned to -135 degrees
- moved R128 99.6 mm to (139.6, 213.3), turned to -135 degrees
- moved R544 97.4 mm to (182.2, 167.0), turned to -15 degrees
- moved C541 94.6 mm to (181.8, 168.4), turned to -15 degrees
- moved C118 89.3 mm to (147.8, 236.0), turned to -45 degrees
- moved R707 84.7 mm to (142.2, 212.3), turned to 45 degrees
- moved C109 79.4 mm to (129.2, 170.0), turned to -90 degrees
- moved C542 79.2 mm to (183.6, 165.8), turned to 75 degrees
- moved C543 78.6 mm to (178.6, 164.9), turned to 75 degrees
- moved R524 75.1 mm to (165.9, 188.9), turned to 45 degrees
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Connections:
- C704 pad 1: VBAT -> VPACK
- C705 pad 1: VBAT -> VPACK
- J102 pad 1: VPACK -> GND
- J102 pad 2: GND -> /Alimentation/PACK_MID
- J103 pad 1: VBAT -> GND
- J103 pad 2: GND -> /Traces et turbine/ESC_SIG
- U501 pad 5: /Capteurs/VREF_RX -> /Capteurs/G_F
- U501 pad 6: /Capteurs/PD_FL -> /Capteurs/FB_F
- U501 pad 7: /Capteurs/TIA_FL -> /Capteurs/AMP_F
- U501 pad 8: /Capteurs/TIA_L -> /Capteurs/U501_SPARE_3
- U501 pad 9: /Capteurs/PD_L -> /Capteurs/U501_SPARE_3
- U502 pad 1: /Capteurs/AMP_F -> /Capteurs/TIA_FL
- U502 pad 10: /Capteurs/G_L -> /Capteurs/VREF_RX
- U502 pad 12: GND -> /Capteurs/VREF_RX
- U502 pad 2: /Capteurs/FB_F -> /Capteurs/PD_FL
- U502 pad 3: /Capteurs/G_F -> /Capteurs/VREF_RX
- U502 pad 8: /Capteurs/AMP_L -> /Capteurs/U502_SPARE_3
- U502 pad 9: /Capteurs/FB_L -> /Capteurs/U502_SPARE_3

Commit message: Réenregistre la carte au format KiCad 10.99 et retouche dix placements
État de travail de l'utilisateur, commité tel quel avant la pose des
règles de conception : passage au format 20260901 du fork (transform,
réglages BOM, réglages DRC nouveaux) et déplacement de C214, C569, C543,
C568, C119, FB101, R546, R545, R547 et C522.

Co-Authored-By: Claude Opus 5.5 <noreply@anthropic.com>
Parts:
- moved R432 346.5 mm to (0.00, 0.00), turned to 0 degrees
- moved C412 345.8 mm to (0.00, 0.00), turned to 0 degrees
- moved R412 343.9 mm to (0.00, 0.00), turned to 0 degrees
- moved D412 343.5 mm to (0.00, 0.00), turned to 0 degrees
- moved U412 343.5 mm to (0.00, 0.00), turned to 0 degrees
- moved R431 343.0 mm to (0.00, 0.00), turned to 0 degrees
- moved R456 342.6 mm to (0.00, 0.00), turned to 0 degrees
- moved C411 342.0 mm to (0.00, 0.00), turned to 0 degrees
- moved R411 340.6 mm to (0.00, 0.00), turned to 0 degrees
- moved D411 339.7 mm to (0.00, 0.00), turned to 0 degrees
- moved U411 339.7 mm to (0.00, 0.00), turned to 0 degrees
- moved R430 338.3 mm to (0.00, 0.00), turned to 0 degrees
- moved R455 338.3 mm to (0.00, 0.00), turned to 0 degrees
- moved C410 337.0 mm to (0.00, 0.00), turned to 0 degrees
- moved R410 336.2 mm to (0.00, 0.00), turned to 0 degrees
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