File: electronics/UsainBot.kicad_pcb (KiCad board)
At the start: 4 copper layers, 155 x 164.9 mm, 343 parts, among them J101 TYPE-C-31-M-12, J102 Pack 2S - AMASS MR30, J103 Montage vertical ESC (prototy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, J201 TC2030-IDC-FP, J301 Moteur Faulhaber + IE2, J351 Moteur Faulhaber + IE2, J601 OLED SSD1306 I2C, J701 Module OTA (ESP32-C3), M1 Faulhaber 1524T006SR + IE2 + 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, M2 Faulhaber 1524T006SR + IE2 + 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, M3 Turbine_EDF27_dessus, Q101 AO3400A, Q102 AO4407A, Q103 AO4407A, Q104 AO3400A, Q401 AO3400A, Q402 AO3400A, Q501 AO3400A, Q521 AO3400A, Q541 AO3400A, Q601 AO3400A, Q602 AO3400A, Q701 SI2301CDS, Q702 AO3400A, SW101 MARCHE / ARRET, SW601 SKRHABE010, SW602 START, SW603 RESET, U101 USBLC6-2SC6, U102 BQ25887RGER, U103 TPS62933DRLR, U105 PCA9685PW, U201 STM32H723ZGT6, U301 DRV8874PWPR, U302 TPS70950DBVR, U351 DRV8874PWPR, U401 ITR8307/S17/TR8(B), U402 ITR8307/S17/TR8(B), U403 ITR8307/S17/TR8(B), U404 ITR8307/S17/TR8(B), U405 ITR8307/S17/TR8(B), U406 ITR8307/S17/TR8(B), U407 ITR8307/S17/TR8(B), U408 ITR8307/S17/TR8(B), U409 ITR8307/S17/TR8(B), U410 ITR8307/S17/TR8(B), U411 ITR8307/S17/TR8(B), U412 ITR8307/S17/TR8(B), U501 TLV9064, U502 TLV9064, U503 LSM6DSOTR, U504 TLV9064, U701 W25Q128JVSIQ, Y201 25 MHz / 10 ppm

Commit message: Update placement
Parts:
- moved SW101 84.0 mm to (211.8, 162.4), turned to 180 degrees
- moved F101 51.6 mm to (140.4, 131.9)
- moved D102 39.5 mm to (189.8, 122.5)
- moved J102 25.9 mm to (142.4, 136.7)
- moved C311 23.3 mm to (97.3, 158.9), turned to 0 degrees
- moved U302 22.6 mm to (93.8, 160.3), turned to 90 degrees
- moved J103 22.2 mm to (166.1, 136.6)
- moved C704 21.5 mm to (165.5, 128.5)
- moved R106 20.1 mm to (111.7, 131.6), turned to 0 degrees
- moved C310 18.4 mm to (94.9, 163.3), turned to 0 degrees
- moved C705 15.5 mm to (159.7, 130.3), turned to 180 degrees
- moved D412 13.4 mm to (209.7, 263.1)
- moved R456 12.6 mm to (212.5, 263.0), turned to 149.715 degrees
- moved C108 8.73 mm to (122.4, 122.7), turned to 90 degrees
- moved C412 8.73 mm to (215.4, 261.3)
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