File: electronics/01-power.kicad_sch (KiCad schematic)
At the start: 57 parts, among them J101 TYPE-C-31-M-12, J102 Pack 2S LiFePO4 (XT30), J103 Equilibrage JST-XH 2S, J104 NTC pack 10k B3435, J105 ON/OFF deporte 10 A, Q101 AO3400A, Q102 AO4407A, U101 USBLC6-2SC6, U102 BQ25887RGER, U103 TPS62933DRLR

Commit message: Passe le microcontrôleur en LQFP144 et lit les deux courants au même instant
Le LQFP100 avait ses seize entrées ADC prises — douze voies de ligne, trois
de télémétrie, une sortie de multiplexeur — et c'est ce multiplexeur qui
posait le vrai problème : il interdisait par construction de lire les deux
courants moteur ensemble. On lisait un moteur, on commutait, on attendait
l'établissement, on lisait l'autre. Le STM32H723ZGT6 en LQFP144 place
PF11 sur ADC1_INP2 et PF13 sur ADC2_INP2 : même numéro de voie sur deux
convertisseurs, donc une lecture simultanée en mode double, et le 74HC4051
disparaît de la carte.

Le brochage étant donné par nom de port et non par numéro de broche, le
passage a coûté deux affectations sur quatre-vingt-sept. Une affectation est
un choix de port — PA0 porte la voie de ligne 00 — jamais un choix de patte.
Une table numérotée aurait demandé de recopier 144 lignes à la main, et une
erreur de brochage ne se voit pas à l'ERC.

Ajoute une huitième feuille, les témoins de ligne. Ce qu'on regarde pendant
un essai n'est pas un témoin d'état générique, c'est ce que voit la
moustache : une LED par capteur, à l'aplomb du capteur qu'elle rapporte, et
un capteur borgne se voit avant la course plutôt qu'après. Le rapport
cyclique suit le signal, sinon rien ne dirait si la ligne est au bord ou au
centre du trait. PCA9685 à l'adresse 0x40 sur I²C2, 52 octets par rafale
soit 1,2 ms à 400 kHz, en DMA hors de la boucle rapide.

Remplace l'interrupteur à glissière par une mise sous tension à bouton
poussoir : une impulsion amorce, le microcontrôleur se tient lui-même, et
c'est lui qui coupe. La glissière demandait une place au bord de carte que
le pack, l'équilibrage et les fils de l'ESC ont fini par prendre — et elle
ne savait pas éteindre proprement, couper le 3,3 V sous les pieds du
firmware n'ayant jamais rien écrit dans la flash.

Ajoute au générateur le contrôle qui manquait : deux extrémités de nets
différents au même point. Il a fallu qu'il relie B+ à B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
Parts:
- removed J103: Equilibrage JST-XH 2S, Connector_JST:JST_XH_B3B-XH-AM_1x03_P2.50mm_Vertical, symbol Connector_Generic:Conn_01x03
- removed J105: ON/OFF deporte 10 A, Connector_JST:JST_VH_B2P-VH_1x02_P3.96mm_Vertical, symbol Connector_Generic:Conn_01x02
- added C122: 100nF, Capacitor_SMD:C_0402_1005Metric, symbol Device:C
- added C123: 1uF, Capacitor_SMD:C_0402_1005Metric, symbol Device:C
- added D106: BAT54, Diode_SMD:D_SOD-323, symbol Device:D_Schottky
- added Q103: AO4407A, Package_SO:SOIC-8_3.9x4.9mm_P1.27mm, symbol Pacabot:AO4407A
- added Q104: AO3400A, Package_TO_SOT_SMD:SOT-23, symbol Transistor_FET:AO3400A
- added R124: 100R, Resistor_SMD:R_0402_1005Metric, symbol Device:R
- added R125: 10k, Resistor_SMD:R_0402_1005Metric, symbol Device:R
- added R126: 100k, Resistor_SMD:R_0402_1005Metric, symbol Device:R
- added R127: 470k, Resistor_SMD:R_0402_1005Metric, symbol Device:R
- added R128: 220k, Resistor_SMD:R_0402_1005Metric, symbol Device:R
- added SW101: MARCHE / ARRET, Button_Switch_SMD:SW_SPST_B3U-1000P, symbol Switch:SW_Push
- C101: value 1uF/25V -> 1uF; Dielectric (none) -> X5R; Voltage (none) -> 25V
- C102, C103, C106, C107: value 22uF/25V -> 22uF; Dielectric (none) -> X5R; Voltage (none) -> 25V
- C104, C110, C113, C114, C115, C118, C120, C121: footprint Capacitor_SMD:C_0603_1608Metric -> Capacitor_SMD:C_0402_1005Metric; Dielectric (none) -> X7R; Voltage (none) -> 25V
- C105: Dielectric (none) -> X5R; Voltage (none) -> 25V
- C108, C111, C112: value 10uF/25V -> 10uF; Dielectric (none) -> X5R; Voltage (none) -> 25V
- C109: value 100uF/16V -> 100uF; Dielectric (none) -> ALU; Voltage (none) -> 16V
- C116, C117: value 22uF/10V -> 22uF; Dielectric (none) -> X5R; Voltage (none) -> 10V
- C119: value 10uF/10V -> 10uF; Dielectric (none) -> X5R; Voltage (none) -> 10V
- F101: value 10 A -> 12 A
- J102: value Pack 2S LiFePO4 (XT30) -> Pack 2S - puissance
- J104: value NTC pack 10k B3435 -> Pack 2S - equilibrage; footprint Connector_JST:JST_PH_B2B-PH-K_1x02_P2.00mm_Vertical -> Connector_JST:JST_XH_B3B-XH-A_1x03_P2.50mm_Vertical; symbol Connector_Generic:Conn_01x02 -> Connector_Generic:Conn_01x03
- R101, R102, R103, R104, R105, R106, R108, R109, R110, R111, R112, R113, R114, R115, R116, R117, R118: footprint Resistor_SMD:R_0603_1608Metric -> Resistor_SMD:R_0402_1005Metric; Power (none) -> 63mW
- R107: value 10R / 1 W -> 10R; footprint Resistor_SMD:R_1206_3216Metric -> Resistor_SMD:R_2512_6332Metric; Power (none) -> 1W
- R119: value 68k -> 22k; footprint Resistor_SMD:R_0603_1608Metric -> Resistor_SMD:R_0402_1005Metric; Power (none) -> 63mW
- R120: value 33k -> 10k; footprint Resistor_SMD:R_0603_1608Metric -> Resistor_SMD:R_0402_1005Metric; Power (none) -> 63mW
Connections:
- net VBAT_SW_OUT is gone; now on net VBAT: Q102.5 (D), Q102.6 (D), Q102.7 (D), Q102.8 (D)
- net GND: now also J104.1 (Pin_1), C122.2, C123.2, Q104.2 (S), R126.2, R128.2, SW101.2; no longer J104.2 (Pin_2), R114.2
- net PACK_MID: now also J104.2 (Pin_2)
- net TS: no longer J104.1 (Pin_1)
- net VBAT: now also Q103.5 (D), Q103.6 (D), Q103.7 (D), Q103.8 (D); no longer Q102.1 (S), Q102.2 (S), Q102.3 (S)
- net VBAT_SW_IN: now also Q102.1 (S), Q102.2 (S), Q102.3 (S), R114.2, Q103.1 (S), Q103.2 (S), Q103.3 (S), R125.1
- net VPACK: now also J104.3 (Pin_3)
- net QREV_G renamed PWR_G
- net PWR_G: now also C123.1, D106.1 (K), Q103.4 (G), Q104.3 (D)
- new net BTN_N: D106.2 (A), R125.2, R127.1, SW101.1
- new net PWR_BTN: C122.1, R127.2, R128.1
- new net PWR_HOLD: R124.1
- new net Q104_G: Q104.1 (G), R124.2, R126.1
Other:
- note added: "7,3 V -> 2,28 V, directement sur PC0. Le 74HC4051 qui multiplexait cette mesure avec les deux IPROPI a disparu avec le passage au LQFP144 : chacun des trois a desormais son entree, et surtout les deux courants moteur se lisent au meme instant (PF11 sur ADC1, PF13 sur ADC2, meme numero de voie). Thevenin 6,9 k, C121 sert de reservoir de charge pour l echantillonnage."
- note added: "D. Pack 2S : puissance et equilibrage, interrupteur general"
- note added: "Le diviseur emule un 103AT a 25 C : la fenetre de temperature est neutralisee, le pack n embarque pas de NTC."
- note added: "Pack : XT30 vertical pour le courant, JST-XH pour la nappe d equilibrage qui apporte le point milieu au BQ25887. Coupure par deux canaux P en parallele (Rds/2), grille rappelee a la source par R114 : coupe par defaut, aucune fuite de grille. MISE SOUS TENSION PAR BOUTON POUSSOIR. L appui tire la grille au 0 V par D106 et les FET conduisent. Le firmware met PE0 a 1 des le demarrage : Q104 tient la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"
- note removed: "7,3 V -> 2,38 V sur ADC3 (PC0)"
- note removed: "Canal P en serie cote haut : drain vers la batterie, source vers la charge. Polarite correcte -> Vgs = -Vbat, le canal conduit. Polarite inversee -> bloque. Une Schottky aurait coute 1,2 W a 3 A."
- note removed: "D. Pack 2S, coupure generale et protection contre l inversion"
- note removed: "Le chargeur est en amont de l interrupteur : le robot se recharge eteint."
- moved on the sheet: C115, C121, F101, Q102, R116, R117, R118, R119, R120

Commit message: Replace la carte autour de ses chaînes analogiques et y intègre le pack commun et l'ESC
Le placement du 4 septembre rangeait les pièces par zone. Celui-ci part des
nets et des vraies pastilles, et affecte chaque condensateur à une broche
plutôt qu'à une couronne autour du boîtier. Le STM32 pivote de 180° sur son
centre pour tourner son côté analogique vers la barrette. Chaque station
laser reçoit son propre TLV9064 (U504 s'ajoute pour la station L), et la
liaison photodiode → TIA tombe de 34, 56 et 69 mm à 3,1, 7,4 et 2,9 mm. La
boucle de retour du TIA passe de 140–150 mm à 3,55. Cinq découplages
suivent : C568, C569/C570 sur VREF_RX, C223/C224 sur VBAT du MCU et C351
sur VREF_MOT du pont droit.

`layout.py`, `layout_fit.json` et `place_pcb.py --reset` ne décrivent plus
cette carte. Le README le dit en tête, et les nouveaux outils partent du
PCB courant, jamais de l'ancienne table. `audit_placement_geometry.py` relit
les courtyards orientés et les contrôle sous Shapely, `placement_metrics.py`
et `preview_analog_paths.py` mesurent distances et couloirs sans poser une
piste. `refine_placement.py` calcule la table, `apply_refined_placement.py`
l'écrit en vérifiant verrous et UUID : il ne se rejoue pas après une
retouche à la main.

L'alimentation change de nature. Le pack LiFePO4 et son ESC sur VBAT
laissent place à un pack 2S commun, chimie encore à choisir, que la carte,
les moteurs et la turbine partagent. Une seule prise MR30 à trois contacts
porte GND, point milieu et VPACK, et remplace XT30 + JST-XH. L'ESC devient
un EMAX Bullet 12A (12 A continu, 15 A crête, sans BEC) sur VPACK brut,
monté debout sur J103. J104 et J702 disparaissent. ESC103 et M703 sont des
symboles hors carte : les phases moteur ne reçoivent aucun pad fictif, et
le module ne compte qu'une fois dans la nomenclature. R107 passe de 10 à
47 Ω pour ramener l'équilibrage à 88 mA et 0,36 W, sous le watt de son
boîtier 2512. La recharge reste inhibée par défaut matériel tant que
cellules, profil et fir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
Parts:
- removed J104: Pack 2S - equilibrage, Connector_JST:JST_XH_B3B-XH-A_1x03_P2.50mm_Vertical, symbol Connector_Generic:Conn_01x03
- J102: value Pack 2S - puissance -> Pack 2S - AMASS MR30; footprint Connector_AMASS:AMASS_XT30U-M_1x02_P5.0mm_Vertical -> Pacabot:AMASS_MR30PB-M_1x03_P3.50mm_Vertical; symbol Connector_Generic:Conn_01x02 -> Connector_Generic:Conn_01x03; Harness (none) -> Project pinout: 1 GND / 2 PACK_MID / 3 VPACK; AWG16 power, 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; MPN (none) -> MR30PB-M30.G.Y; Manufacturer (none) -> AMASS; Mating_connector (none) -> MR30-F.G.Y; optional cover 98023.PG; Mechanical_revision (none) -> AMASS MR30PB-M 2021V1: 11.9x5.3x10.4mm; 3mm tails; pitch3.5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; Operating_budget (none) -> ESC 12A continuous /15A peak + 2 DC motors x1A + electronic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; Rated_current (none) -> 20 A per manufacturer at deltaT 85K with AWG16; thermal val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
- R107: value 10R -> 47R
Connections:
- net GND: now also J102.1 (Pin_1); no longer J102.2 (Pin_2)
- net PACK_MID: now also J102.2 (Pin_2)
- net VPACK: now also J102.3 (Pin_3); no longer J102.1 (Pin_1)
Other:
- note added: "CD haut = charge inhibee par defaut materiel. Pack commun 2S : cellules / capacite / chimie non choisies. Definir VCELLREG, courant, protections et firmware AVANT toute charge. Le programme de charge reste a implementer et a valider."
- note added: "Mesure VBAT : diviseur 22k / 10k, directement sur PC0. Le 74HC4051 qui multiplexait cette mesure avec les deux IPROPI a disparu avec le passage au LQFP144 : chacun des trois a desormais son entree, et surtout les deux courants moteur se lisent au meme instant (PF11 sur ADC1, PF13 sur ADC2, meme numero de voie). Thevenin 6,9 k, C121 sert de reservoir de charge pour l echantillonnage."
- note added: "Pack commun : J102 MR30 3 contacts GND / MID / VPACK. MID alimente la mesure / equilibrage du BQ25887. Coupure par deux canaux P en parallele (Rds/2), grille rappelee a la source par R114 : coupe par defaut, aucune fuite de grille. MISE SOUS TENSION PAR BOUTON POUSSOIR. L appui tire la grille au 0 V par D106 et les FET conduisent. Le firmware met PE0 a 1 des le demarrage : Q104 tient la grille, l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"
- note added: "R107 = 47R / 1W : equilibrage ~88mA a 4,2V; dissipation ~0,36W. Maximum conservateur a 4,6V : 0,46W avec tolerance 1%; verifier thermique. BQ25887 : equilibrage qualifie au-dessus de 3,7V/cellule (Li-ion/LiPo)."
- note removed: "7,3 V -> 2,28 V, directement sur PC0. Le 74HC4051 qui multiplexait cette mesure avec les deux IPROPI a disparu avec le passage au LQFP144 : chacun des trois a desormais son entree, et surtout les deux courants moteur se lisent au meme instant (PF11 sur ADC1, PF13 sur ADC2, meme numero de voie). Thevenin 6,9 k, C121 sert de reservoir de charge pour l echantillonnage."
- note removed: "CD haut = charge inhibee. La grille est au 0 V tant que le MCU n a pas ecrit VCELLREG : un pack LiFePO4 ne voit jamais le profil Li-ion par defaut (4,2 V/cellule), meme carte eteinte."
- note removed: "Pack : XT30 vertical pour le courant, JST-XH pour la nappe d equilibrage qui apporte le point milieu au BQ25887. Coupure par deux canaux P en parallele (Rds/2), grille rappelee a la source par R114 : coupe par defaut, aucune fuite de grille. MISE SOUS TENSION PAR BOUTON POUSSOIR. L appui tire la grille au 0 V par D106 et les FET conduisent. Le firmware met PE0 a 1 des le demarrage : Q104 tient la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"
- note removed: "R107 fixe le courant d equilibrage (400 mA max)."

Commit message: Alimente les codeurs en 5 V, renomme les paires USB et passe les résistances des LED en 0603
- Codeurs IE2 : U302 TPS70950 sur VBAT (EN sur +3V3, le 5 V suit le MCU
  dont les entrées FT_h ne tolèrent 5 V qu'alimentées), C310 1 µF et
  C311 4,7 µF ; net /Moteurs/ENC_5V vers J301.4 et J351.4, classe
  ALIM_LOGIQUE. Symbole Pacabot:TPS70950DBV ajouté à la bibliothèque.
- Paires USB : USB_D_P/N et /Alimentation/USB_C_D_P/N, reconnues comme
  paires par KiCad et par le routeur de paires du fork.
- R615, R617, R618 en 0603 à 390/560/560 ohms (≈ 10 mA, ≤ 50 mW à 7,3 V) ;
  R615 et R618 recalées, D609 décalée de 0,25 mm, R617 déplacée à côté
  de R306 faute de place pour une 0603 près de D608.

Schéma et carte concordent pastille par pastille (netlist KiCad 10.0.1) ;
ERC 0, DRC sans nouvelle violation. Détail dans rules-review/README.md.

Co-Authored-By: Claude Opus 5.5 <noreply@anthropic.com>
Connections:
- net USB_DM renamed USB_D_N
- net USB_DM_C renamed USB_C_D_N
- net USB_DP renamed USB_D_P
- net USB_DP_C renamed USB_C_D_P
Changed lines of the file:
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@@
 		)
 	)
-	(label "USB_DP_C"
+	(label "USB_C_D_P"
 		(at 64.77 67.31 0)
 		(fields_autoplaced yes)
@@
 		)
 	)
-	(label "USB_DM_C"
+	(label "USB_C_D_N"
 		(at 64.77 62.23 0)
 		(fields_autoplaced yes)
@@
 		)
 	)
-	(label "USB_DP_C"
+	(label "USB_C_D_P"
 		(at 120.65 44.45 180)
 		(fields_autoplaced yes)
@@
 		)
 	)
-	(global_label "USB_DP"
+	(global_label "USB_D_P"
 		(shape bidirectional)
 		(at 135.89 44.45 0)
@@
 		)
 	)
-	(label "USB_DM_C"
+	(label "USB_C_D_N"
 		(at 120.65 46.99 180)
 		(fields_autoplaced yes)
@@
 		)
 	)
-	(global_label "USB_DM"
+	(global_label "USB_D_N"
 		(shape bidirectional)
 		(at 135.89 46.99 0)
