File: electronics/01-power.kicad_sch (KiCad schematic)
At the start: 65 parts, among them J101 TYPE-C-31-M-12, J102 Pack 2S - AMASS MR30, Q101 AO3400A, Q102 AO4407A, Q103 AO4407A, Q104 AO3400A, SW101 MARCHE / ARRET, U101 USBLC6-2SC6, U102 BQ25887RGER, U103 TPS62933DRLR

Commit message: Update placement
Other:
- moved on the sheet: R114, SW101
