File: electronics/06-hmi.kicad_sch (KiCad schematic)
At the start: 29 parts, among them J601 OLED SSD1306 I2C, J602 Jack de depart, Q601 AO3400A, SW601 TS-006 ou equivalent, SW602 START

Commit message: Passe le microcontrôleur en LQFP144 et lit les deux courants au même instant
Le LQFP100 avait ses seize entrées ADC prises — douze voies de ligne, trois
de télémétrie, une sortie de multiplexeur — et c'est ce multiplexeur qui
posait le vrai problème : il interdisait par construction de lire les deux
courants moteur ensemble. On lisait un moteur, on commutait, on attendait
l'établissement, on lisait l'autre. Le STM32H723ZGT6 en LQFP144 place
PF11 sur ADC1_INP2 et PF13 sur ADC2_INP2 : même numéro de voie sur deux
convertisseurs, donc une lecture simultanée en mode double, et le 74HC4051
disparaît de la carte.

Le brochage étant donné par nom de port et non par numéro de broche, le
passage a coûté deux affectations sur quatre-vingt-sept. Une affectation est
un choix de port — PA0 porte la voie de ligne 00 — jamais un choix de patte.
Une table numérotée aurait demandé de recopier 144 lignes à la main, et une
erreur de brochage ne se voit pas à l'ERC.

Ajoute une huitième feuille, les témoins de ligne. Ce qu'on regarde pendant
un essai n'est pas un témoin d'état générique, c'est ce que voit la
moustache : une LED par capteur, à l'aplomb du capteur qu'elle rapporte, et
un capteur borgne se voit avant la course plutôt qu'après. Le rapport
cyclique suit le signal, sinon rien ne dirait si la ligne est au bord ou au
centre du trait. PCA9685 à l'adresse 0x40 sur I²C2, 52 octets par rafale
soit 1,2 ms à 400 kHz, en DMA hors de la boucle rapide.

Remplace l'interrupteur à glissière par une mise sous tension à bouton
poussoir : une impulsion amorce, le microcontrôleur se tient lui-même, et
c'est lui qui coupe. La glissière demandait une place au bord de carte que
le pack, l'équilibrage et les fils de l'ESC ont fini par prendre — et elle
ne savait pas éteindre proprement, couper le 3,3 V sous les pieds du
firmware n'ayant jamais rien écrit dans la flash.

Ajoute au générateur le contrôle qui manquait : deux extrémités de nets
différents au même point. Il a fallu qu'il relie B+ à B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
Parts:
- removed D602: verte - etat, LED_SMD:LED_0603_1608Metric, symbol Device:LED
- removed D603: rouge - defaut, LED_SMD:LED_0603_1608Metric, symbol Device:LED
- removed D604: jaune - libre, LED_SMD:LED_0603_1608Metric, symbol Device:LED
- removed J602: Jack de depart, Connector_PinHeader_2.54mm:PinHeader_1x02_P2.54mm_Vertical, symbol Connector_Generic:Conn_01x02
- removed R611, R612, R613: 1k, Resistor_SMD:R_0603_1608Metric, symbol Device:R
- added C607: 100nF, Capacitor_SMD:C_0402_1005Metric, symbol Device:C
- added D606: bleue - nez, LED_SMD:LED_0603_1608Metric, symbol Device:LED
- added D608: rouge - coin arriere gauche, LED_SMD:LED_0603_1608Metric, symbol Device:LED
- added D609: rouge - coin arriere droit, LED_SMD:LED_0603_1608Metric, symbol Device:LED
- added D610: BAT54, Diode_SMD:D_SOD-323, symbol Device:D_Schottky
- added Q602: AO3400A, Package_TO_SOT_SMD:SOT-23, symbol Transistor_FET:AO3400A
- added R615: 220R, Resistor_SMD:R_0402_1005Metric, symbol Device:R
- added R617, R618: 300R, Resistor_SMD:R_0402_1005Metric, symbol Device:R
- added R619: 100R, Resistor_SMD:R_0402_1005Metric, symbol Device:R
- added R620: 100k, Resistor_SMD:R_0402_1005Metric, symbol Device:R
- C601, C602, C603, C604, C605, C606: footprint Capacitor_SMD:C_0603_1608Metric -> Capacitor_SMD:C_0402_1005Metric; Dielectric (none) -> X7R; Voltage (none) -> 25V
- J601: footprint Connector_PinHeader_2.54mm:PinHeader_1x04_P2.54mm_Vertical -> Pacabot:OLED_096_I2C
- R601, R602, R603, R604, R605, R606, R607, R608, R609, R610: footprint Resistor_SMD:R_0603_1608Metric -> Resistor_SMD:R_0402_1005Metric; Power (none) -> 63mW
- SW601: value TS-006 ou equivalent -> SKRHABE010; footprint (none) -> Pacabot:SKRHABE010; LCSC (none) -> C144855
Connections:
- net BUZZER: now also C607.1; no longer R609.1
- net GND: now also D610.2 (A), Q602.2 (S), R620.2
- new net BZAC: C607.2, D610.1 (K), R609.1
- new net D606_A: D606.2 (A), R615.2
- new net D608_A: D608.2 (A), R617.2
- new net D609_A: D609.2 (A), R618.2
- new net Q602_G: Q602.1 (G), R619.2, R620.1
- new net TRACK_EN: R619.1
- new net TRACK_SW: D606.1 (K), D608.1 (K), D609.1 (K), Q602.3 (D)
- new net VBAT: R615.1, R617.1, R618.1
Other:
- note added: "Alps SKRHABE010, joystick 4 directions + appui central, 7,35 x 7,5 mm. Contacts A-D vers UP/RIGHT/DOWN/LEFT : l affectation reelle des directions se recale au firmware."
- note added: "Deux des trois bleues du nez ont ete rendues le 4 septembre : il en reste une sur l axe. Avec les deux rouges des coins arriere, la camera a toujours un triangle - position ET cap - et le nez, qui est la partie la plus etroite et la plus chargee de la carte, y gagne deux LED et deux resistances de place."
- note added: "Le bouton suffit au reglement, le geste devant le telemetre n en est qu un complement (machine a etats du firmware)."
- note added: "Plus de temoins d etat generiques : les trois LED verte / rouge / jaune et leurs trois GPIO ont ete rendus le 4 septembre. Ce qu on regarde pendant un essai, c est la barrette - chaque capteur de ligne a maintenant sa LED (feuille 04). Le temoin " BLE alimente " visible du jury reste cable sur le rail +3V3_BLE lui-meme (feuille 07) : il ne peut pas mentir sur l etat reel du module."
- note added: "Roue libre obligatoire (bobine) ; grille couplee en alternatif : un GPIO fige ne peut pas laisser 200 mA en continu dans le buzzer."
- note added: "Suivi camera - 1 bleue au nez, 2 rouges aux coins arriere"
- note removed: "Bouton et jack en parallele : les deux moyens que le reglement enumere sont cables, le geste devant le telemetre n en est qu un complement (voir la machine a etats du firmware)."
- note removed: "Diode de roue libre obligatoire : la bobine du buzzer renvoie sa surtension dans le drain."
- note removed: "Empreinte a confirmer sur la reference retenue (LCSC C3674) : commun unique cote masse, cinq contacts au repos ouverts."
- note removed: "Le temoin " BLE alimente " visible du jury est cable sur le rail +3V3_BLE lui-meme (feuille 07) : il ne peut pas mentir sur l etat reel de l alimentation du module."
- note removed: "Temoins"
- moved on the sheet: Q601, R609, R610

Commit message: Alimente les codeurs en 5 V, renomme les paires USB et passe les résistances des LED en 0603
- Codeurs IE2 : U302 TPS70950 sur VBAT (EN sur +3V3, le 5 V suit le MCU
  dont les entrées FT_h ne tolèrent 5 V qu'alimentées), C310 1 µF et
  C311 4,7 µF ; net /Moteurs/ENC_5V vers J301.4 et J351.4, classe
  ALIM_LOGIQUE. Symbole Pacabot:TPS70950DBV ajouté à la bibliothèque.
- Paires USB : USB_D_P/N et /Alimentation/USB_C_D_P/N, reconnues comme
  paires par KiCad et par le routeur de paires du fork.
- R615, R617, R618 en 0603 à 390/560/560 ohms (≈ 10 mA, ≤ 50 mW à 7,3 V) ;
  R615 et R618 recalées, D609 décalée de 0,25 mm, R617 déplacée à côté
  de R306 faute de place pour une 0603 près de D608.

Schéma et carte concordent pastille par pastille (netlist KiCad 10.0.1) ;
ERC 0, DRC sans nouvelle violation. Détail dans rules-review/README.md.

Co-Authored-By: Claude Opus 5.5 <noreply@anthropic.com>
Parts:
- R615: value 220R -> 390R; footprint Resistor_SMD:R_0402_1005Metric -> Resistor_SMD:R_0603_1608Metric; Power 63mW -> 100mW
- R617, R618: value 300R -> 560R; footprint Resistor_SMD:R_0402_1005Metric -> Resistor_SMD:R_0603_1608Metric; Power 63mW -> 100mW
Changed lines of the file:
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@@
 			)
 		)
-		(property "Value" "220R"
+		(property "Value" "390R"
 			(at 40.3 113.27 0)
 			(effects
@@
 			)
 		)
-		(property "Footprint" "Resistor_SMD:R_0402_1005Metric"
+		(property "Footprint" "Resistor_SMD:R_0603_1608Metric"
 			(at 38.1 113.03 0)
 			(effects
@@
 			)
 		)
-		(property "Power" "63mW"
+		(property "Power" "100mW"
 			(at 40.3 115.81 0)
 			(effects
@@
 			)
 		)
-		(property "Value" "300R"
+		(property "Value" "560R"
 			(at 70.3 113.27 0)
 			(effects
@@
 			)
 		)
-		(property "Footprint" "Resistor_SMD:R_0402_1005Metric"
+		(property "Footprint" "Resistor_SMD:R_0603_1608Metric"
 			(at 68.58 113.03 0)
 			(effects
@@
 			)
 		)
-		(property "Power" "63mW"
+		(property "Power" "100mW"
 			(at 70.3 115.81 0)
 			(effects
@@
 			)
 		)
-		(property "Value" "300R"
+		(property "Value" "560R"
 			(at 100.3 113.27 0)
 			(effects
@@
 			)
 		)
-		(property "Footprint" "Resistor_SMD:R_0402_1005Metric"
+		(property "Footprint" "Resistor_SMD:R_0603_1608Metric"
 			(at 97.79 113.03 0)
 			(effects
@@
 			)
 		)
-		(property "Power" "63mW"
+		(property "Power" "100mW"
 			(at 100.3 115.81 0)
 			(effects
