File: electronics/03-motors.kicad_sch (KiCad schematic)
At the start: 39 parts, among them J301 Moteur gauche + encodeur, J351 Moteur droit + encodeur, U301 DRV8874PWPR, U351 DRV8874PWPR

Commit message: Passe le microcontrôleur en LQFP144 et lit les deux courants au même instant
Le LQFP100 avait ses seize entrées ADC prises — douze voies de ligne, trois
de télémétrie, une sortie de multiplexeur — et c'est ce multiplexeur qui
posait le vrai problème : il interdisait par construction de lire les deux
courants moteur ensemble. On lisait un moteur, on commutait, on attendait
l'établissement, on lisait l'autre. Le STM32H723ZGT6 en LQFP144 place
PF11 sur ADC1_INP2 et PF13 sur ADC2_INP2 : même numéro de voie sur deux
convertisseurs, donc une lecture simultanée en mode double, et le 74HC4051
disparaît de la carte.

Le brochage étant donné par nom de port et non par numéro de broche, le
passage a coûté deux affectations sur quatre-vingt-sept. Une affectation est
un choix de port — PA0 porte la voie de ligne 00 — jamais un choix de patte.
Une table numérotée aurait demandé de recopier 144 lignes à la main, et une
erreur de brochage ne se voit pas à l'ERC.

Ajoute une huitième feuille, les témoins de ligne. Ce qu'on regarde pendant
un essai n'est pas un témoin d'état générique, c'est ce que voit la
moustache : une LED par capteur, à l'aplomb du capteur qu'elle rapporte, et
un capteur borgne se voit avant la course plutôt qu'après. Le rapport
cyclique suit le signal, sinon rien ne dirait si la ligne est au bord ou au
centre du trait. PCA9685 à l'adresse 0x40 sur I²C2, 52 octets par rafale
soit 1,2 ms à 400 kHz, en DMA hors de la boucle rapide.

Remplace l'interrupteur à glissière par une mise sous tension à bouton
poussoir : une impulsion amorce, le microcontrôleur se tient lui-même, et
c'est lui qui coupe. La glissière demandait une place au bord de carte que
le pack, l'équilibrage et les fils de l'ESC ont fini par prendre — et elle
ne savait pas éteindre proprement, couper le 3,3 V sous les pieds du
firmware n'ayant jamais rien écrit dans la flash.

Ajoute au générateur le contrôle qui manquait : deux extrémités de nets
différents au même point. Il a fallu qu'il relie B+ à B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
Parts:
- C301, C302, C303, C305, C306, C308, C309, C352, C353, C355, C356, C358, C359: footprint Capacitor_SMD:C_0603_1608Metric -> Capacitor_SMD:C_0402_1005Metric; Dielectric (none) -> X7R; Voltage (none) -> 25V
- C304, C354: value 100uF/16V -> 100uF; footprint Capacitor_SMD:CP_Elec_6.3x7.7 -> Capacitor_Tantalum_SMD:CP_EIA-7343-20_Kemet-V; Dielectric (none) -> X5R; Voltage (none) -> 16V poly
- C307, C357: value 100nF / X7R 50 V -> 100nF; Dielectric (none) -> X7R; Voltage (none) -> 50V
- J301: value Moteur gauche + encodeur -> Moteur Faulhaber + IE2; footprint Connector_JST:JST_PH_B6B-PH-K_1x06_P2.00mm_Vertical -> Connector_TE-Connectivity:TE_Micro-MaTch_215079-6_2x03_P1.27mm_Vertical; symbol Connector_Generic:Conn_01x06 -> Pacabot:Motor_Faulhaber; MPN (none) -> TE 7-215079-6
- J351: value Moteur droit + encodeur -> Moteur Faulhaber + IE2; footprint Connector_JST:JST_PH_B6B-PH-K_1x06_P2.00mm_Vertical -> Connector_TE-Connectivity:TE_Micro-MaTch_215079-6_2x03_P1.27mm_Vertical; symbol Connector_Generic:Conn_01x06 -> Pacabot:Motor_Faulhaber; MPN (none) -> TE 7-215079-6
- R301, R302, R303, R304, R305, R306, R307, R308, R309, R310, R353, R354, R355, R356, R357, R358, R359, R360: footprint Resistor_SMD:R_0603_1608Metric -> Resistor_SMD:R_0402_1005Metric; Power (none) -> 63mW
Connections:
- net +3V3: now also J301.4 (VDD), J351.4 (VDD); no longer J301.3 (Pin_3), J351.3 (Pin_3)
- net ENC_L_A_RAW: now also J301.6 (A); no longer J301.5 (Pin_5)
- net ENC_L_B_RAW: now also J301.5 (B); no longer J301.6 (Pin_6)
- net ENC_R_A_RAW: now also J351.6 (A); no longer J351.5 (Pin_5)
- net ENC_R_B_RAW: now also J351.5 (B); no longer J351.6 (Pin_6)
- net GND: now also J301.3 (GND), J351.3 (GND); no longer J301.4 (Pin_4), J351.4 (Pin_4)
- net MOT_L_OUT1: now also J301.2 (M+); no longer J301.1 (Pin_1)
- net MOT_L_OUT2: now also J301.1 (M-); no longer J301.2 (Pin_2)
- net MOT_R_OUT1: now also J351.2 (M+); no longer J351.1 (Pin_1)
- net MOT_R_OUT2: now also J351.1 (M-); no longer J351.2 (Pin_2)
Other:
- note added: "Nappe Faulhaber sur Micro-MaTch 215079-6 : impairs a gauche, fil rouge = M+. Fils moteur torsades, 100 nF aux bornes."
- note removed: "Fils moteur torsades, 100 nF aux bornes. Filtre d entree du timer active en plus du RC."
- moved on the sheet: C308, C309, C358, C359, J301, J351, R309, R310, R359, R360

Commit message: Replace la carte autour de ses chaînes analogiques et y intègre le pack commun et l'ESC
Le placement du 4 septembre rangeait les pièces par zone. Celui-ci part des
nets et des vraies pastilles, et affecte chaque condensateur à une broche
plutôt qu'à une couronne autour du boîtier. Le STM32 pivote de 180° sur son
centre pour tourner son côté analogique vers la barrette. Chaque station
laser reçoit son propre TLV9064 (U504 s'ajoute pour la station L), et la
liaison photodiode → TIA tombe de 34, 56 et 69 mm à 3,1, 7,4 et 2,9 mm. La
boucle de retour du TIA passe de 140–150 mm à 3,55. Cinq découplages
suivent : C568, C569/C570 sur VREF_RX, C223/C224 sur VBAT du MCU et C351
sur VREF_MOT du pont droit.

`layout.py`, `layout_fit.json` et `place_pcb.py --reset` ne décrivent plus
cette carte. Le README le dit en tête, et les nouveaux outils partent du
PCB courant, jamais de l'ancienne table. `audit_placement_geometry.py` relit
les courtyards orientés et les contrôle sous Shapely, `placement_metrics.py`
et `preview_analog_paths.py` mesurent distances et couloirs sans poser une
piste. `refine_placement.py` calcule la table, `apply_refined_placement.py`
l'écrit en vérifiant verrous et UUID : il ne se rejoue pas après une
retouche à la main.

L'alimentation change de nature. Le pack LiFePO4 et son ESC sur VBAT
laissent place à un pack 2S commun, chimie encore à choisir, que la carte,
les moteurs et la turbine partagent. Une seule prise MR30 à trois contacts
porte GND, point milieu et VPACK, et remplace XT30 + JST-XH. L'ESC devient
un EMAX Bullet 12A (12 A continu, 15 A crête, sans BEC) sur VPACK brut,
monté debout sur J103. J104 et J702 disparaissent. ESC103 et M703 sont des
symboles hors carte : les phases moteur ne reçoivent aucun pad fictif, et
le module ne compte qu'une fois dans la nomenclature. R107 passe de 10 à
47 Ω pour ramener l'équilibrage à 88 mA et 0,36 W, sous le watt de son
boîtier 2512. La recharge reste inhibée par défaut matériel tant que
cellules, profil et fir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
Parts:
- added C351: 100nF, Capacitor_SMD:C_0402_1005Metric, symbol Device:C
Connections:
- net GND: now also C351.2
- net VREF_MOT: now also C351.1
Other:
- note added: "C301 au pied de U301.5 ; C351 au pied de U351.5. Le rail commun de seuil est filtre localement aux deux ponts."
Changed lines of the file:
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@@
 	)
 	(embedded_fonts no)
+	(symbol
+		(lib_id "Device:C")
+		(at 250.19 270.51 0)
+		(unit 1)
+		(exclude_from_sim no)
+		(in_bom yes)
+		(on_board yes)
+		(dnp no)
+		(property "Reference" "C351"
+			(at 252.3 267.46 0)
+			(effects
+				(font
+					(size 1 1)
+				)
+				(justify left)
+			)
+		)
+		(property "Value" "100nF"
+			(at 252.3 270 0)
+			(effects
+				(font
+					(size 1 1)
+				)
+				(justify left)
+			)
+		)
+		(property "Footprint" "Capacitor_SMD:C_0402_1005Metric"
+			(at 250.19 270.51 0)
+			(effects
+				(font
+					(size 1 1)
+				)
+				(justify left)
+				(hide yes)
+			)
+		)
+		(property "Datasheet" "~"
+			(at 250.19 270.51 0)
+			(effects
+				(font
+					(size 1 1)
+				)
+				(justify left)
+				(hide yes)
+			)
+		)
+		(property "Description" ""
+			(at 250.19 270.51 0)
+			(effects
+				(font
+					(size 1 1)
+				)
+				(justify left)
+				(hide yes)
+			)
+		)
+		(property "Voltage" "25V"
+			(at 252.3 272.54 0)
+			(effects
+				(font
+					(size 1 1)
+				)
+				(justify left)
+			)
+		)
+		(property "Dielectric" "X7R"
+			(at 252.3 275.08 0)
+			(effects
+				(font
+					(size 1 1)
+				)
+				(justify left)
+				(hide yes)
+			)
+		)
+		(pin "1"
+		)
+		(pin "2"
+		)
+		(instances
+			(project "UsainBot"
+				(path "/e216f09c-2662-6258-2b51-4f4f498f79d0/f091e242-b2d2-a8c1-4ba0-334789aaf38f"
+					(reference "C351")
+					(unit 1)
+				)
+			)
+		)
+	)
+	(wire
+		(pts
+			(xy 250.19 266.7)
+			(xy 250.19 264.16)
+		)
+		(stroke
+			(width 0)
+			(type default)
+		)
+	)
+	(label "VREF_MOT"
+		(at 250.19 264.16 0)
+		(fields_autoplaced yes)
+		(effects
+			(font
+				(size 1 1)
+			)
+			(justify left bottom)
+		)
+	)
+	(wire
+		(pts
+			(xy 250.19 274.32)
+			(xy 250.19 276.86)
+		)
+		(stroke
+			(width 0)
+			(type default)
+		)
+	)
+	(symbol
+		(lib_id "power:GND")
+		(at 250.19 276.86 0)
+		(unit 1)
+		(exclude_from_sim no)
+		(in_bom no)
+		(on_board yes)
+		(dnp no)
+		(property "Reference" "#PWR9201"
+			(at 250.19 267.97 0)
+			(effects
+				(font
+					(size 1 1)
+				)
+				(hide yes)
+			)
+		)
+		(property "Value" "GND"
+			(at 250.19 285.75 0)
+			(effects
+				(font
+					(size 1 1)
+				)
+				(hide yes)
+			)
+		)
+		(property "Footprint" ""
+			(at 250.19 276.86 0)
+			(effects
+				(font
+					(size 1 1)
+				)
+				(hide yes)
+			)
+		)
+		(property "Datasheet" "~"
+			(at 250.19 276.86 0)
+			(effects
+				(font
+					(size 1 1)
+				)
+				(hide yes)
+			)
+		)
+		(property "Description" ""
+			(at 250.19 276.86 0)
+			(effects
+				(font
+					(size 1 1)
+				)
+				(hide yes)
+			)
+		)
+		(pin "1"
+		)
+		(instances
+			(project "UsainBot"
+				(path "/e216f09c-2662-6258-2b51-4f4f498f79d0/f091e242-b2d2-a8c1-4ba0-334789aaf38f"
+					(reference "#PWR9201")
+					(unit 1)
+				)
+			)
+		)
+	)
+	(text "C301 au pied de U301.5 ; C351 au pied de U351.5.\nLe rail commun de seuil est filtre localement aux deux ponts."
+		(exclude_from_sim no)
+		(at 70 276 0)
+		(effects
+			(font
+				(size 1 1)
+			)
+			(justify left bottom)
+		)
+	)
 )

Commit message: Alimente les codeurs en 5 V, renomme les paires USB et passe les résistances des LED en 0603
- Codeurs IE2 : U302 TPS70950 sur VBAT (EN sur +3V3, le 5 V suit le MCU
  dont les entrées FT_h ne tolèrent 5 V qu'alimentées), C310 1 µF et
  C311 4,7 µF ; net /Moteurs/ENC_5V vers J301.4 et J351.4, classe
  ALIM_LOGIQUE. Symbole Pacabot:TPS70950DBV ajouté à la bibliothèque.
- Paires USB : USB_D_P/N et /Alimentation/USB_C_D_P/N, reconnues comme
  paires par KiCad et par le routeur de paires du fork.
- R615, R617, R618 en 0603 à 390/560/560 ohms (≈ 10 mA, ≤ 50 mW à 7,3 V) ;
  R615 et R618 recalées, D609 décalée de 0,25 mm, R617 déplacée à côté
  de R306 faute de place pour une 0603 près de D608.

Schéma et carte concordent pastille par pastille (netlist KiCad 10.0.1) ;
ERC 0, DRC sans nouvelle violation. Détail dans rules-review/README.md.

Co-Authored-By: Claude Opus 5.5 <noreply@anthropic.com>
Parts:
- added C310: 1uF, Capacitor_SMD:C_0402_1005Metric, symbol Device:C
- added C311: 4.7uF, Capacitor_SMD:C_0603_1608Metric, symbol Device:C
- added U302: TPS70950DBVR, Package_TO_SOT_SMD:SOT-23-5, symbol Pacabot:TPS70950DBV
Connections:
- net +3V3: now also U302.3 (EN); no longer J301.4 (VDD), J351.4 (VDD)
- net GND: now also C310.2, C311.2, U302.2 (GND)
- net VBAT: now also C310.1, U302.1 (IN)
- new net ENC_5V: C311.1, J301.4 (VDD), J351.4 (VDD), U302.5 (OUT)
- no-connect marks 0 -> 1
Other:
- note added: "Codeurs IE2 : 4,5-5,5 V (Faulhaber). EN sur +3V3 : le 5 V n'apparaît qu'avec le MCU, dont PB4/PB5/PC6/PC7 (FT_h) ne tolèrent 5 V qu'alimentés. 26 mA max, chute <= 0,26 V."

Commit message: Retire les pièces abandonnées et ouvre le schéma dans le fork 10.99
- Bibliothèque : retrait du GM12-N20 (empreinte, générateur, STEP, roues
  Pololu), de l'ESC Multistar, du XT30, de l'inter Shouhan et de
  ITR8307_dessous, qu'aucune feuille ni la carte n'utilisent plus.
- firmware/UsainBot.ioc retiré : il configurait un STM32G431 LQFP32, pas
  le H723ZGT6 de la carte. mechanics/motorM20 et motorHolder (ère N20)
  retirés.
- Feuille racine : sheet_instances réduit à "/" ; le fork 10.99 refusait
  le schéma (« malformed root sheet instance path »). ERC 0 en 10.0.1,
  aucune violation hors configuration de bibliothèques en 10.99.
- Cartouche moteurs : Faulhaber 1524 et codeurs IE2 au lieu du GM12-N20.
- UsainBot.pdf régénéré (il datait du 6 septembre).
- README et kicad-lib/README remis à jour : LQFP144, Faulhaber, BPV10NF,
  MR30, garde au sol, points ouverts (pack 2S, ESC prototype).

Co-Authored-By: Claude Opus 5.5 <noreply@anthropic.com>
Other:
- title: UsainBot - Ponts en H DRV8874, moteurs GM12-N20 et encodeurs -> UsainBot - Ponts en H DRV8874, moteurs Faulhaber 1524 et codeurs IE2
Changed lines of the file:
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@@
 	(paper "A3")
 	(title_block
-		(title "UsainBot - Ponts en H DRV8874, moteurs GM12-N20 et encodeurs")
+		(title "UsainBot - Ponts en H DRV8874, moteurs Faulhaber 1524 et codeurs IE2")
 		(date "2026-08-30")
 		(rev "A")
